File: central_control.sch (KiCad schematic (older format))
At the start: 6 parts

Commit message: Finish sheets
Parts:
- added C?: 100n, symbol Device:C
- added C?: 2u2 16V, symbol Device:C
- added C?: 22u, symbol Device:C
- added H? (x2): MountingHole, symbol Mechanical:MountingHole
- added J?: SWD, symbol Connector:Conn_01x05_Female
- added J?: POWER, symbol Connector:Conn_01x02_Female
- added J?: UART, symbol Connector:Conn_01x02_Female
- added J?: SPI, symbol Connector:Conn_01x03_Female
- added J?: I2C, symbol Connector:Conn_01x02_Female
- added J?: ADC, symbol Connector:Conn_01x04_Female
- added J?: PWM, symbol Connector:Conn_01x04_Female
- added J? (x3): 3V3, symbol Connector:Conn_01x02_Female
- added L?: L_Small, symbol Device:L_Small
- added R?: 4k7, symbol Device:R
- added R?: 1k5, symbol Device:R
- added SW?: SW_Push, symbol Switch:SW_Push
- added U?: TPS62175DQC, Package_SON:WSON-10-1EP_2x3mm_P0.5mm_EP0.84x2.4mm_ThermalVias, symbol Regulator_Switching:TPS62175DQC
Connections:
- net labels added: ADC1_IN0, ADC1_IN1, ADC1_IN2, ADC1_IN3, SPI1_MISO, SPI1_MOSI, SPI1_SCK, TIM3_CH1, TIM3_CH2, TIM3_CH3, TIM3_CH4, USART1_RX, USART1_TX, Vdrive, ~RST
- wire segments 42 -> 139
- no-connect marks 0 -> 7
Other:
- note added: "MCU with reset circuit"
- note added: "PCB mounting holes"
- note added: "connectors"
- note added: "decoupling"
- note added: "max. 28V"
- note added: "step down converter for MCU"
- moved on the sheet: C?

Commit message: Replace MCU and add CAN Flexible Datarate. Close #1
Parts:
- removed C? (x4): 100n, symbol Device:C
- removed SW?: SW_Push, symbol Switch:SW_Push
- removed U?: STM32L071K8Ux, Package_DFN_QFN:QFN-32-1EP_5x5mm_P0.5mm_EP3.45x3.45mm, symbol MCU_ST_STM32L0:STM32L071K8Ux
- added J?: CAN, symbol Connector:Conn_01x02_Female
- added J?: 3V3, symbol Connector:Conn_01x02_Female
- added U?: STM32G0C1KCU, symbol extraSymbols:STM32G0C1KxU
Connections:
- net labels added: FDCAN1_RX, FDCAN1_TX, SPI3_MISO, SPI3_MOSI, SPI3_SCK
- net labels removed: SPI1_MISO, SPI1_MOSI, SPI1_SCK
- wire segments 139 -> 107
- no-connect marks 7 -> 11
Other:
- note added: "MCU (reset circuit not needed in G0 series)"
- note removed: "MCU with reset circuit"
- note removed: "decoupling"
- moved on the sheet: C?, H?

Commit message: Add EEPROM for configuration's sake
Parts:
- added C?: 100n, symbol Device:C
- added R? (x2): 2k, symbol Device:R
- added U?: 24LC64, Package_TO_SOT_SMD:SOT-23-5, symbol extraSymbols:24LC64
Connections:
- wire segments 107 -> 130
Other:
- note added: "EEPROM for configuration"
- note added: "Extern transceiver needed!"
Changed lines of the file:
@@
 Text Label 10300 1150 2    50   ~ 0
 FDCAN1_TX
+Text Notes 9850 850  0    47   ~ 0
+Extern transceiver needed!
+Text Label 4150 4350 2    50   ~ 0
+I2C1_SCL
+Text Label 4150 4550 2    50   ~ 0
+I2C1_SDA
+$Comp
+L extraSymbols:24LC64 U?
+U 1 1 602DEC51
+P 4850 4500
+F 0 "U?" H 4850 4915 50  0000 C CNN
+F 1 "24LC64" H 4850 4824 50  0000 C CNN
+F 2 "Package_TO_SOT_SMD:SOT-23-5" H 4850 4500 50  0001 C CNN
+F 3 "" H 4850 4500 50  0001 C CNN
+	1    4850 4500
+	1    0    0    -1
+$EndComp
+$Comp
+L Device:C C?
+U 1 1 602E6B83
+P 5400 4750
+F 0 "C?" H 5450 4850 50  0000 L CNN
+F 1 "100n" H 5450 4650 50  0000 L CNN
+F 2 "" H 5438 4600 50  0001 C CNN
+F 3 "~" H 5400 4750 50  0001 C CNN
+	1    5400 4750
+	1    0    0    -1
+$EndComp
+$Comp
+L power:+3.3V #PWR?
+U 1 1 602E6DA5
+P 5400 4500
+F 0 "#PWR?" H 5400 4350 50  0001 C CNN
+F 1 "+3.3V" H 5415 4673 50  0000 C CNN
+F 2 "" H 5400 4500 50  0001 C CNN
+F 3 "" H 5400 4500 50  0001 C CNN
+	1    5400 4500
+	1    0    0    -1
+$EndComp
+$Comp
+L power:GND #PWR?
+U 1 1 602E6F57
+P 4850 5000
+F 0 "#PWR?" H 4850 4750 50  0001 C CNN
+F 1 "GND" H 4855 4827 50  0000 C CNN
+F 2 "" H 4850 5000 50  0001 C CNN
+F 3 "" H 4850 5000 50  0001 C CNN
+	1    4850 5000
+	1    0    0    -1
+$EndComp
+Wire Wire Line
+	5200 4550 5400 4550
+Wire Wire Line
+	5400 4550 5400 4500
+Wire Wire Line
+	5400 4550 5400 4600
+Connection ~ 5400 4550
+$Comp
+L Device:R R?
+U 1 1 602F88ED
+P 4200 4100
+F 0 "R?" V 4200 4050 50  0000 L CNN
+F 1 "2k" V 4300 4050 50  0000 L CNN
+F 2 "" V 4130 4100 50  0001 C CNN
+F 3 "~" H 4200 4100 50  0001 C CNN
+	1    4200 4100
+	1    0    0    -1
+$EndComp
+$Comp
+L Device:R R?
+U 1 1 602F8BDB
+P 4400 4100
+F 0 "R?" V 4400 4050 50  0000 L CNN
+F 1 "2k" V 4500 4050 50  0000 L CNN
+F 2 "" V 4330 4100 50  0001 C CNN
+F 3 "~" H 4400 4100 50  0001 C CNN
+	1    4400 4100
+	1    0    0    -1
+$EndComp
+Wire Wire Line
+	4200 4250 4200 4350
+Wire Wire Line
+	4200 4350 4150 4350
+Wire Wire Line
+	4200 4350 4500 4350
+Connection ~ 4200 4350
+Wire Wire Line
+	4400 4250 4400 4550
+Wire Wire Line
+	4400 4550 4150 4550
+Wire Wire Line
+	4400 4550 4500 4550
+Connection ~ 4400 4550
+$Comp
+L power:+3.3V #PWR?
+U 1 1 6030A91E
+P 4300 3850
+F 0 "#PWR?" H 4300 3700 50  0001 C CNN
+F 1 "+3.3V" H 4315 4023 50  0000 C CNN
+F 2 "" H 4300 3850 50  0001 C CNN
+F 3 "" H 4300 3850 50  0001 C CNN
+	1    4300 3850
+	1    0    0    -1
+$EndComp
+Wire Wire Line
+	4300 3850 4300 3900
+Wire Wire Line
+	4300 3900 4200 3900
+Wire Wire Line
+	4200 3900 4200 3950
+Wire Wire Line
+	4300 3900 4400 3900
+Wire Wire Line
+	4400 3900 4400 3950
+Connection ~ 4300 3900
+Wire Wire Line
+	4450 4450 4500 4450
+Wire Wire Line
+	5400 4950 5400 4900
+Wire Wire Line
+	4450 4950 4850 4950
+Wire Wire Line
+	4450 4450 4450 4950
+Wire Wire Line
+	4850 5000 4850 4950
+Connection ~ 4850 4950
+Wire Wire Line
+	4850 4950 5250 4950
+Wire Wire Line
+	5200 4350 5250 4350
+Wire Wire Line
+	5250 4350 5250 4950
+Connection ~ 5250 4950
+Wire Wire Line
+	5250 4950 5400 4950
+Wire Notes Line
+	3750 5250 5700 5250
+Wire Notes Line
+	5700 5250 5700 3600
+Wire Notes Line
+	5700 3600 3750 3600
+Wire Notes Line
+	3750 3600 3750 5250
+Text Notes 3750 3550 0    50   ~ 0
+EEPROM for configuration
 $EndSCHEMATC

Commit message: Add voltage dividers for temperature measurement and optional connector for poti
Parts:
- removed J? (x4): 3V3, symbol Connector:Conn_01x02_Female
- added C? (x4): 100n, symbol Device:C
- added J?: POTI, symbol Connector:Conn_01x03_Female
- added R? (x4): 10k, symbol Device:R
- J? (x3): symbol Connector:Conn_01x02_Female -> Connector:Conn_01x04_Female
- J?: symbol Connector:Conn_01x03_Female -> Connector:Conn_01x05_Female
- J?: symbol Connector:Conn_01x04_Female -> Connector:Conn_01x05_Female
Connections:
- net labels added: ADC1_IN4, TEMP0, TEMP1, TEMP2, TEMP3
- wire segments 130 -> 165
- no-connect marks 11 -> 10
Other:
- note added: "External\ntransceiver needed!"
- note added: "like ST-Link v2"
- note added: "voltage dividers for NTC\nall NTCs will be connected to 3V3"
- note removed: "Extern transceiver needed!"
- moved on the sheet: H?, J?

Commit message: Replace MCU again (with STM32L431KB) STM32G0B1 is not available on digikey/mouser
Parts:
- removed C?: 10u, symbol Device:C
- removed U?: STM32G0C1KCU, symbol extraSymbols:STM32G0C1KxU
- added C? (x2): 100n, symbol Device:C
- added C?: 10u, symbol Device:C
- added C?: 10n, symbol Device:C_Small
- added C?: 1u, symbol Device:C_Small
- added FB?: Ferrite_Bead_Small, symbol Device:Ferrite_Bead_Small
- added JP?: SolderJumper_2_Open, symbol Jumper:SolderJumper_2_Open
- added SW?: SW_Push, symbol Switch:SW_Push
- added U?: STM32L431KBUx, Package_DFN_QFN:QFN-32-1EP_5x5mm_P0.5mm_EP3.45x3.45mm, symbol MCU_ST_STM32L4:STM32L431KBUx
- J?: symbol Connector:Conn_01x05_Female -> Connector:Conn_01x06_Female
Connections:
- net labels added: ADC1_IN11, ADC1_IN12, ADC1_IN15, ADC1_IN16, ADC1_IN9, CAN1_RX, CAN1_TX, SPI1_MISO, SPI1_MOSI, SPI1_SCK, SWO, TIM2_CH1, TIM2_CH2, TIM2_CH3, TIM2_CH4
- net labels removed: ADC1_IN0, ADC1_IN1, ADC1_IN2, ADC1_IN3, ADC1_IN4, FDCAN1_RX, FDCAN1_TX, SPI3_MISO, SPI3_MOSI, SPI3_SCK, TIM3_CH1, TIM3_CH2, TIM3_CH3, TIM3_CH4
- wire segments 165 -> 208
- no-connect marks 10 -> 5
Other:
- note added: "(BOOT0)"
- note added: "MCU (with reset circuit and decoupling capacitors)"
- note removed: "MCU (reset circuit not needed in G0 series)"
- moved on the sheet: C?, R?

Commit message: Update MCU
Parts:
- U?: value STM32L431KBUx -> STM32L432KBUx; symbol MCU_ST_STM32L4:STM32L431KBUx -> MCU_ST_STM32L4:STM32L432KBUx
Changed lines of the file:
@@
 	9750 750  9750 2100
 $Comp
-L MCU_ST_STM32L4:STM32L431KBUx U?
+L MCU_ST_STM32L4:STM32L432KBUx U?
 U 1 1 6031DCAC
 P 2600 4200
 F 0 "U?" H 2950 5050 50  0000 C CNN
-F 1 "STM32L431KBUx" V 2600 4150 50  0000 C CNN
+F 1 "STM32L432KBUx" V 2600 4150 50  0000 C CNN
 F 2 "Package_DFN_QFN:QFN-32-1EP_5x5mm_P0.5mm_EP3.45x3.45mm" H 2200 3300 50  0001 R CNN
-F 3 "http://www.st.com/st-web-ui/static/active/en/resource/technical/document/datasheet/DM00257211.pdf" H 2600 4200 50  0001 C CNN
+F 3 "http://www.st.com/st-web-ui/static/active/en/resource/technical/document/datasheet/DM00257205.pdf" H 2600 4200 50  0001 C CNN
 	1    2600 4200
 	1    0    0    -1

Commit message: Annotate sheets and assign symbols
Parts:
- removed J?: ADC, symbol Connector:Conn_01x05_Female
- removed J?: PWM, symbol Connector:Conn_01x04_Female
- added J10: PLED1, Connector_Molex:Molex_PicoBlade_53047-0310_1x03_P1.25mm_Vertical, symbol Connector:Conn_01x03_Female
- added J11: PLED3, Connector_Molex:Molex_PicoBlade_53047-0310_1x03_P1.25mm_Vertical, symbol Connector:Conn_01x03_Female
- added J8: PLED0, Connector_Molex:Molex_PicoBlade_53047-0310_1x03_P1.25mm_Vertical, symbol Connector:Conn_01x03_Female
- added J9: PLED2, Connector_Molex:Molex_PicoBlade_53047-0310_1x03_P1.25mm_Vertical, symbol Connector:Conn_01x03_Female
- C10, C12: renamed from C?; footprint (none) -> Capacitor_SMD:C_0805_2012Metric
- C11, C13, C14, C15, C16, C17, C18, C19, C7, C8, C9: renamed from C?; footprint (none) -> Capacitor_SMD:C_0603_1608Metric
- FB1: renamed from FB?; footprint (none) -> Resistor_SMD:R_0603_1608Metric
- H1, H2: renamed from H?; footprint (none) -> MountingHole:MountingHole_2.7mm_M2.5_ISO14580
- J12: renamed from J?; footprint (none) -> Connector_PinHeader_2.54mm:PinHeader_1x06_P2.54mm_Vertical
- J13: renamed from J?; footprint (none) -> Connector_PinHeader_2.54mm:PinHeader_1x03_P2.54mm_Vertical
- J14, J6, J7: renamed from J?; footprint (none) -> Connector_PinHeader_2.54mm:PinHeader_1x04_P2.54mm_Vertical
- J4: renamed from J?; footprint (none) -> Connector_Molex:Molex_PicoBlade_53047-0210_1x02_P1.25mm_Vertical
- J5: renamed from J?; footprint (none) -> Connector_PinHeader_2.54mm:PinHeader_1x05_P2.54mm_Vertical
- JP2: renamed from JP?; footprint (none) -> Jumper:SolderJumper-2_P1.3mm_Open_TrianglePad1.0x1.5mm
- L2: renamed from L?; value L_Small -> 10u; footprint (none) -> Inductor_SMD:L_1210_3225Metric
- R10, R11, R12, R13, R6, R7, R8, R9: renamed from R?; footprint (none) -> Resistor_SMD:R_0603_1608Metric
- SW1: renamed from SW?; footprint (none) -> extraFootprints:PTS636_F-leads
- gave numbers to parts that had none: 3
Connections:
- net +3V3: now also J10.1 (Pin_1), J11.1 (Pin_1), J8.1 (Pin_1), J9.1 (Pin_1)
- net ADC1_IN11: now also J10.2 (Pin_2)
- net ADC1_IN12: now also J9.2 (Pin_2)
- net ADC1_IN15: now also J11.2 (Pin_2)
- net ADC1_IN9: now also J8.2 (Pin_2)
- net TIM2_CH1: now also J8.3 (Pin_3)
- net TIM2_CH2: now also J10.3 (Pin_3)
- net TIM2_CH3: now also J9.3 (Pin_3)
- net TIM2_CH4: now also J11.3 (Pin_3)

Commit message: Split project into individual projects and reannotate sheets
Parts:
- renumbered C7 to C1, C16 to C10, C17 to C11, C18 to C12, C19 to C13, C8 to C2, C9 to C3, C10 to C4, C11 to C5, C12 to C6, C13 to C7, C14 to C8, C15 to C9, J4 to J1, J13 to J10, J14 to J11, J5 to J2, J6 to J3, J7 to J4, J8 to J5, J9 to J6, J10 to J7, J11 to J8, J12 to J9, JP2 to JP1, L2 to L1, R6 to R1, R7 to R2, R8 to R3, R9 to R4, R10 to R5, R11 to R6, R12 to R7, R13 to R8, U2 to U1, U3 to U2, U4 to U3
