File: high_power_LED.sch (KiCad schematic (older format))
At the start: 0 parts

Commit message: Finish sheets
Parts:
- added D? (x3): LED_PAD, symbol Device:LED_PAD
- added H? (x2): MountingHole, symbol Mechanical:MountingHole
- added HS?: Heatsink_Pad, symbol Mechanical:Heatsink_Pad
- added J?: Anode, symbol Connector:Conn_01x01_Female
- added J?: TH+, symbol Connector:Conn_01x01_Female
- added J?: TH-, symbol Connector:Conn_01x01_Female
- added J?: Cathode, symbol Connector:Conn_01x01_Female
- added JP? (x3): SolderJumper_2_Open, symbol Jumper:SolderJumper_2_Open
- added TH?: Thermistor, symbol Device:Thermistor
Connections:
- new net: D?.1 (K), D?.2 (A), JP?.1 (A), JP?.2 (B) (x2)
- new net: D?.2 (A), J?.1 (Pin_1), JP?.1 (A)
- new net: D?.3 (PAD), D?.3 (PAD), D?.3 (PAD), HS?.1
- new net: D?.1 (K), J?.1 (Pin_1), JP?.2 (B)
- new net: J?.1 (Pin_1), TH?.1
- new net: J?.1 (Pin_1), TH?.2
Other:
- note added: "high power LED"
- note added: "temperature measurement"
- note added: "you can skip LEDs by soldering it's jumper pad"
