File: solder_workspace_lighting.sch (KiCad schematic (older format))
At the start: 0 parts

Commit message: Finish sheets
Other:
- note added: "each sheet stands for a single pcb"
Changed lines of the file:
@@
 F1 "high_power_LED.sch" 50
 $EndSheet
+Text Notes 4750 5200 0    79   ~ 0
+each sheet stands for a single pcb
 $EndSCHEMATC
