File: high_power_LED.kicad_pcb (KiCad board)
At the start: 2 copper layers, 0 parts

Commit message: Finish high power led pcb
Parts:
- added D1: LED_PAD, extraFootprints:Cree-XLamp-MX6, F.Cu at (126.5, 104.1)
- added D2: LED_PAD, extraFootprints:Cree-XLamp-MX6, F.Cu at (134.9, 104.1)
- added D3: LED_PAD, extraFootprints:Cree-XLamp-MX6, F.Cu at (143.3, 104.1)
- added H1: MountingHole, MountingHole:MountingHole_2.7mm_M2.5_ISO14580, F.Cu at (124.1, 94.1)
- added H2: MountingHole, MountingHole:MountingHole_2.7mm_M2.5_ISO14580, F.Cu at (145.7, 113.7)
- added HS1: Heatsink_Pad, Heatsink:Heatsink_AAVID_573300D00010G_TO-263, B.Cu at (134.9, 104.1)
- added J1: LED, Connector_PinHeader_2.54mm:PinHeader_1x02_P2.54mm_Vertical, B.Cu at (133.9, 113.5)
- added J2: TH, Connector_Molex:Molex_PicoBlade_53047-0210_1x02_P1.25mm_Vertical, B.Cu at (128.0, 113.3)
- added JP1: SolderJumper_2_Open, Jumper:SolderJumper-2_P1.3mm_Open_TrianglePad1.0x1.5mm, F.Cu at (122.4, 104.1)
- added JP2: SolderJumper_2_Open, Jumper:SolderJumper-2_P1.3mm_Open_TrianglePad1.0x1.5mm, F.Cu at (130.8, 104.1)
- added JP3: SolderJumper_2_Open, Jumper:SolderJumper-2_P1.3mm_Open_TrianglePad1.0x1.5mm, F.Cu at (139.2, 104.1)
- added TH1: Thermistor, Resistor_SMD:R_0603_1608Metric, B.Cu at (134.9, 105.9)
- added svg2mod: G***, extraFootprints:netz39-logo, B.Cu at (129.8, 94.0)
Routing:
- net /Cathode: track 0.00 -> 27.9 mm
- net Net-(D2-Pad1): track 0.00 -> 20.8 mm
- net Net-(D1-Pad1): track 0.00 -> 16.4 mm
- net /Anode: track 0.00 -> 15.0 mm
- net /TH+: track 0.00 -> 10.4 mm
- net /TH-: track 0.00 -> 10.0 mm
- net Net-(D1-Pad3): vias 0 -> 11
- added copper zone on B.Cu, net Net-(D1-Pad3)
- added copper zone on F.Cu, net Net-(D1-Pad3)
Other:
- board outline added: 27.9 x 25.9 mm
- board text added: "high power LED pcb v1.0 by Max Grau 2021-03"
