File: constant_current_source/constant_current_source.kicad_pcb (KiCad board)
At the start: 2 copper layers, 0 parts

Commit message: Finish constant current source pcb
Parts:
- added C1: 100n, Capacitor_SMD:C_0603_1608Metric, B.Cu at (146.4, 112.8)
- added C2: 10u 16V, Capacitor_SMD:C_0805_2012Metric, F.Cu at (139.8, 122.6)
- added C3: 2u2 16V, Capacitor_SMD:C_0603_1608Metric, F.Cu at (141.7, 122.3)
- added C4: 3n3, Capacitor_SMD:C_0603_1608Metric, B.Cu at (142.5, 111.9)
- added C5: 220n, Capacitor_SMD:C_0603_1608Metric, F.Cu at (144.1, 121.7)
- added C6: 2u2 16V, Capacitor_SMD:C_0603_1608Metric, F.Cu at (147.6, 118.5)
- added D1: MBR0520L, Diode_SMD:D_SOD-123, F.Cu at (152.0, 123.1)
- added J1: Conn, Connector_Molex:Molex_PicoBlade_53047-0410_1x04_P1.25mm_Vertical, F.Cu at (152.8, 117.5)
- added J2: LED, Connector_PinHeader_2.54mm:PinHeader_1x02_P2.54mm_Vertical, B.Cu at (134.9, 117.1)
- added JP1: SolderJumper_2_Open, Jumper:SolderJumper-2_P1.3mm_Open_TrianglePad1.0x1.5mm, F.Cu at (148.3, 114.8)
- added L1: 3u3, Inductor_SMD:L_Abracon_ASPI-3012S, F.Cu at (147.6, 122.2)
- added Q1: IRLML0030, Package_TO_SOT_SMD:SOT-23, F.Cu at (138.6, 115.4)
- added R1: 10k, Resistor_SMD:R_0603_1608Metric, F.Cu at (148.8, 112.0)
- added R2: 10k, Resistor_SMD:R_0603_1608Metric, F.Cu at (147.2, 112.0)
- added R3: 4k7, Resistor_SMD:R_0603_1608Metric, B.Cu at (144.5, 109.5)
- added R4: 2k, Resistor_SMD:R_0603_1608Metric, B.Cu at (141.4, 109.5)
- added R5: 10k, Resistor_SMD:R_0603_1608Metric, F.Cu at (144.8, 111.1)
- added U1: LT3474, Package_SO:TSSOP-16-1EP_4.4x5mm_P0.65mm, F.Cu at (143.5, 115.6)
- added svg2mod: G***, extraFootprints:netz39-logo, B.Cu at (146.4, 114.3)
Routing:
- net /VIN: track 0.00 -> 27.2 mm, vias 0 -> 2
- net /PWM: track 0.00 -> 26.2 mm
- net /Anode: track 0.00 -> 16.5 mm
- net Net-(C5-Pad2): track 0.00 -> 11.6 mm
- net /SHDN: track 0.00 -> 10.4 mm
- net GND: track 0.00 -> 9.35 mm, vias 0 -> 27
- net Net-(R3-Pad2): track 0.00 -> 5.33 mm, vias 0 -> 1
- net Net-(C4-Pad2): track 0.00 -> 4.96 mm, vias 0 -> 1
- net Net-(C6-Pad1): track 0.00 -> 3.77 mm, vias 0 -> 5
- net Net-(R3-Pad1): track 0.00 -> 3.65 mm, vias 0 -> 1
- net Net-(C5-Pad1): track 0.00 -> 3.50 mm
- net /Cathode: track 0.00 -> 3.37 mm
- net Net-(C1-Pad2): track 0.00 -> 2.00 mm, vias 0 -> 1
- net Net-(R2-Pad1): track 0.00 -> 1.42 mm
- added copper zone on B.Cu, net GND
- added copper zone on F.Cu, net GND
- added copper zone on B.Cu, net Net-(C6-Pad1)
- added copper zone on F.Cu, net Net-(C6-Pad1)
Other:
- board outline added: 22.9 x 15.9 mm
- board text added: "constant current source v1.0 by Max Grau 2021-03"
