File: central_control/central_control.kicad_pcb (KiCad board)
At the start: 2 copper layers, 0 parts

Commit message: Finish central control PCB
Parts:
- added C1: 100n, Capacitor_SMD:C_0603_1608Metric, B.Cu at (174.9, 79.8)
- added C10: 100n, Capacitor_SMD:C_0603_1608Metric, B.Cu at (165.4, 78.0)
- added C11: 100n, Capacitor_SMD:C_0603_1608Metric, B.Cu at (177.8, 84.3)
- added C12: 100n, Capacitor_SMD:C_0603_1608Metric, B.Cu at (167.6, 80.3)
- added C13: 100n, Capacitor_SMD:C_0603_1608Metric, B.Cu at (177.8, 77.2)
- added C2: 2u2 16V, Capacitor_SMD:C_0603_1608Metric, F.Cu at (169.3, 61.8)
- added C3: 100n, Capacitor_SMD:C_0603_1608Metric, B.Cu at (171.6, 75.6)
- added C4: 10u, Capacitor_SMD:C_0805_2012Metric, B.Cu at (171.1, 72.8)
- added C5: 100n, Capacitor_SMD:C_0603_1608Metric, F.Cu at (166.4, 74.3)
- added C6: 22u, Capacitor_SMD:C_0805_2012Metric, F.Cu at (171.8, 64.9)
- added C7: 1u, Capacitor_SMD:C_0603_1608Metric, B.Cu at (168.4, 76.5)
- added C8: 10n, Capacitor_SMD:C_0603_1608Metric, B.Cu at (168.4, 78.0)
- added C9: 100n, Capacitor_SMD:C_0603_1608Metric, F.Cu at (172.0, 83.6)
- added FB1: Ferrite_Bead_Small, Resistor_SMD:R_0603_1608Metric, B.Cu at (168.4, 74.9)
- added H1: MountingHole, MountingHole:MountingHole_2.7mm_M2.5_ISO14580, F.Cu at (183.1, 63.8)
- added H2: MountingHole, MountingHole:MountingHole_2.7mm_M2.5_ISO14580, F.Cu at (161.5, 88.4)
- added J1: POWER, Connector_Molex:Molex_PicoBlade_53047-0210_1x02_P1.25mm_Vertical, F.Cu at (164.8, 58.2)
- added J10: POTI, Connector_Molex:Molex_PicoBlade_53047-0310_1x03_P1.25mm_Vertical, F.Cu at (169.4, 88.4)
- added J11: CAN, Connector_Molex:Molex_PicoBlade_53047-0410_1x04_P1.25mm_Vertical, F.Cu at (183.1, 69.6)
- added J2: SPI, Connector_Molex:Molex_PicoBlade_53047-0510_1x05_P1.25mm_Vertical, F.Cu at (178.6, 58.2)
- added J3: UART, Connector_Molex:Molex_PicoBlade_53047-0410_1x04_P1.25mm_Vertical, F.Cu at (170.5, 58.2)
- added J4: I2C, Connector_Molex:Molex_PicoBlade_53047-0410_1x04_P1.25mm_Vertical, F.Cu at (177.5, 88.4)
- added J5: PLED0, Connector_Molex:Molex_PicoBlade_53047-0310_1x03_P1.25mm_Vertical, F.Cu at (161.5, 76.7)
- added J6: PLED2, Connector_Molex:Molex_PicoBlade_53047-0310_1x03_P1.25mm_Vertical, F.Cu at (183.1, 84.6)
- added J7: PLED1, Connector_Molex:Molex_PicoBlade_53047-0310_1x03_P1.25mm_Vertical, F.Cu at (161.5, 83.5)
- added J8: PLED3, Connector_Molex:Molex_PicoBlade_53047-0310_1x03_P1.25mm_Vertical, F.Cu at (183.1, 77.7)
- added J9: SWD, Connector_PinHeader_2.54mm:PinHeader_1x06_P2.54mm_Vertical, F.Cu at (160.8, 57.4)
- added JP1: SolderJumper_2_Open, Jumper:SolderJumper-2_P1.3mm_Open_TrianglePad1.0x1.5mm, F.Cu at (178.8, 75.4)
- added L1: 10u, Inductor_SMD:L_1210_3225Metric, F.Cu at (170.1, 67.7)
- added R1: 4k7, Resistor_SMD:R_0603_1608Metric, F.Cu at (163.7, 64.4)
- added R2: 1k5, Resistor_SMD:R_0603_1608Metric, F.Cu at (165.4, 64.4)
- added R3: 2k, Resistor_SMD:R_0603_1608Metric, F.Cu at (179.2, 81.0)
- added R4: 2k, Resistor_SMD:R_0603_1608Metric, F.Cu at (177.5, 81.0)
- added R5: 10k, Resistor_SMD:R_0603_1608Metric, B.Cu at (165.4, 76.5)
- added R6: 10k, Resistor_SMD:R_0603_1608Metric, B.Cu at (179.3, 84.3)
- added R7: 10k, Resistor_SMD:R_0603_1608Metric, B.Cu at (166.1, 80.3)
- added R8: 10k, Resistor_SMD:R_0603_1608Metric, B.Cu at (179.3, 77.2)
- added SW1: SW_Push, extraFootprints:PTS636_F-leads, F.Cu at (167.6, 80.6)
- added U1: TPS62175DQC, Package_SON:WSON-10-1EP_2x3mm_P0.5mm_EP0.84x2.4mm_ThermalVias, F.Cu at (168.0, 64.3)
- added U2: STM32L432KBUx, Package_DFN_QFN:QFN-32-1EP_5x5mm_P0.5mm_EP3.45x3.45mm, F.Cu at (173.2, 77.7)
- added U3: 24LC64, Package_TO_SOT_SMD:SOT-23-5, F.Cu at (174.8, 83.8)
- added svg2mod: G***, extraFootprints:netz39-logo, B.Cu at (175.3, 64.0)
Routing:
- net +3V3: track 0.00 -> 150.4 mm, vias 0 -> 8
- net GND: track 0.00 -> 49.1 mm, vias 0 -> 49
- net /SPI1_SCK: track 0.00 -> 33.8 mm, vias 0 -> 2
- net /SWDCLK: track 0.00 -> 27.5 mm, vias 0 -> 2
- net /SWDIO: track 0.00 -> 24.7 mm, vias 0 -> 4
- net /USART1_RX: track 0.00 -> 21.0 mm, vias 0 -> 1
- net /SPI1_MOSI: track 0.00 -> 20.8 mm, vias 0 -> 2
- net /USART1_TX: track 0.00 -> 20.6 mm, vias 0 -> 1
- net /TIM2_CH4: track 0.00 -> 20.4 mm
- net /SPI1_MISO: track 0.00 -> 20.1 mm
- net /I2C1_SCL: track 0.00 -> 20.1 mm, vias 0 -> 3
- net /I2C1_SDA: track 0.00 -> 19.9 mm, vias 0 -> 1
- net /TIM2_CH3: track 0.00 -> 19.3 mm
- net /SWO: track 0.00 -> 18.5 mm, vias 0 -> 3
- net /~RST: track 0.00 -> 16.3 mm, vias 0 -> 2
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- added copper zone on B.Cu, net GND
- added copper zone on F.Cu, net GND
Other:
- board outline added: 27.3 x 36.2 mm
- board text added: "LED central control v1.0 by Max Grau 2021-03"
