File: central_control/central_control.sch (KiCad schematic (older format))
At the start: 41 parts, among them J1 POWER, J10 POTI, J11 CAN, J2 SPI, J3 UART, J4 I2C, J5 PLED0, J6 PLED2, J7 PLED1, J8 PLED3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

Commit message: Finish central control PCB
Parts:
- J10: footprint Connector_PinHeader_2.54mm:PinHeader_1x03_P2.54mm_Vertical -> Connector_Molex:Molex_PicoBlade_53047-0310_1x03_P1.25mm_Vertical
- J11, J3, J4: footprint Connector_PinHeader_2.54mm:PinHeader_1x04_P2.54mm_Vertical -> Connector_Molex:Molex_PicoBlade_53047-0410_1x04_P1.25mm_Vertical
- J2: footprint Connector_PinHeader_2.54mm:PinHeader_1x05_P2.54mm_Vertical -> Connector_Molex:Molex_PicoBlade_53047-0510_1x05_P1.25mm_Vertical
Connections:
- net ADC1_IN12: now also J10.2 (Pin_2); no longer C11.1, J6.2 (Pin_2), R6.1
- net ADC1_IN15: now also C11.1, J6.2 (Pin_2), R6.1; no longer C13.1, J8.2 (Pin_2), R8.1
- net ADC1_IN16: now also C13.1, J8.2 (Pin_2), R8.1; no longer J10.2 (Pin_2)
Changed lines of the file:
@@
 F 0 "J3" H 6028 1026 50  0000 L CNN
 F 1 "UART" H 6028 935 50  0000 L CNN
-F 2 "Connector_PinHeader_2.54mm:PinHeader_1x04_P2.54mm_Vertical" H 6000 1050 50  0001 C CNN
+F 2 "Connector_Molex:Molex_PicoBlade_53047-0410_1x04_P1.25mm_Vertical" H 6000 1050 50  0001 C CNN
 F 3 "~" H 6000 1050 50  0001 C CNN
 	1    6000 1050
@@
 F 0 "J2" H 5128 1176 50  0000 L CNN
 F 1 "SPI" H 5128 1085 50  0000 L CNN
-F 2 "Connector_PinHeader_2.54mm:PinHeader_1x05_P2.54mm_Vertical" H 5100 1150 50  0001 C CNN
+F 2 "Connector_Molex:Molex_PicoBlade_53047-0510_1x05_P1.25mm_Vertical" H 5100 1150 50  0001 C CNN
 F 3 "~" H 5100 1150 50  0001 C CNN
 	1    5100 1150
@@
 F 0 "J4" H 6928 1026 50  0000 L CNN
 F 1 "I2C" H 6928 935 50  0000 L CNN
-F 2 "Connector_PinHeader_2.54mm:PinHeader_1x04_P2.54mm_Vertical" H 6900 1050 50  0001 C CNN
+F 2 "Connector_Molex:Molex_PicoBlade_53047-0410_1x04_P1.25mm_Vertical" H 6900 1050 50  0001 C CNN
 F 3 "~" H 6900 1050 50  0001 C CNN
 	1    6900 1050
@@
 F 0 "J11" H 10478 1026 50  0000 L CNN
 F 1 "CAN" H 10478 935 50  0000 L CNN
-F 2 "Connector_PinHeader_2.54mm:PinHeader_1x04_P2.54mm_Vertical" H 10450 1050 50  0001 C CNN
+F 2 "Connector_Molex:Molex_PicoBlade_53047-0410_1x04_P1.25mm_Vertical" H 10450 1050 50  0001 C CNN
 F 3 "~" H 10450 1050 50  0001 C CNN
 	1    10450 1050
@@
 Text Label 6800 4500 1    50   ~ 0
 TEMP3
-Text Label 7050 4550 0    50   ~ 0
+Text Label 6250 4550 0    50   ~ 0
 ADC1_IN15
 Text Label 6000 4500 1    50   ~ 0
@@
 	1    0    0    -1
 $EndComp
-Text Label 6250 4550 0    50   ~ 0
+Text Label 10150 1850 2    50   ~ 0
 ADC1_IN12
 Wire Notes Line
@@
 Text Label 8400 1400 2    50   ~ 0
 TEMP3
-Text Label 10150 1850 2    50   ~ 0
+Text Label 7050 4550 0    50   ~ 0
 ADC1_IN16
 Wire Wire Line
@@
 F 0 "J10" H 10428 1826 50  0000 L CNN
 F 1 "POTI" H 10428 1735 50  0000 L CNN
-F 2 "Connector_PinHeader_2.54mm:PinHeader_1x03_P2.54mm_Vertical" H 10400 1850 50  0001 C CNN
+F 2 "Connector_Molex:Molex_PicoBlade_53047-0310_1x03_P1.25mm_Vertical" H 10400 1850 50  0001 C CNN
 F 3 "~" H 10400 1850 50  0001 C CNN
 	1    10400 1850
@@
 Wire Wire Line
 	8400 900  8450 900
-Text Notes 7000 3200 0    50   ~ 0
-voltage dividers for NTC\nall NTCs will be connected to 3V3
 $Comp
 L Connector:Conn_01x03_Female J6
